File: hardware/electronics/source/esp32_self_balancing_robot.kicad_pcb (KiCad board)
At the start: 2 copper layers, 80 x 66 mm, 36 parts, among them J1 ESP32-S3-DevKitC, J2 MPU6050_Breakout, J3 MPM3610_Breakout, J4 DRV8833_Breakout, J5 LEFT_MOTOR, J6 RIGHT_MOTOR, Q1 BC337, Q2 BC337

Commit message: fix: electronic design layouts
Other:
- board text added: "150"
- board text removed: "22"
Changed lines of the file:
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@@
 		)
 	)
-	(gr_text "220"
+	(gr_text "150"
 		(at 191.840634 95.988823 0)
 		(layer "F.SilkS")
@@
 		)
 	)
-	(gr_text "22"
+	(gr_text "47"
 		(at 238.781178 90.38828 0)
 		(layer "F.SilkS")
@@
 		)
 	)
-	(gr_text "22"
+	(gr_text "47"
 		(at 242.619943 90.38828 0)
 		(layer "F.SilkS")
