File: hardware/electronics/source/esp32_self_balancing_robot.kicad_sch (KiCad schematic)
At the start: 29 parts, among them J1 ESP32-S3-DevKitC, J2 MPU6050_Breakout, J3 MPM3610_Breakout, J4 DRV8833_Breakout, J5 LEFT_MOTOR, J6 RIGHT_MOTOR, Q1 BC337, Q2 BC337

Commit message: fix: electronic design layouts
Parts:
- R5: value 220 -> 150
- R7, R8: value 22 -> 47
Changed lines of the file:
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@@
 	(title_block
 		(title "ESP32-S3 SELF BALANCING ROBOT")
+		(date "2026-09-16")
 		(rev "v1.0")
 		(company "Arthur Lawson")
@@
 			)
 		)
-		(property "Value" "22"
+		(property "Value" "47"
 			(at 207.01 26.924 0)
 			(show_name no)
@@
 			)
 		)
-		(property "Value" "22"
+		(property "Value" "47"
 			(at 207.01 21.844 0)
 			(show_name no)
@@
 			)
 		)
-		(property "Value" "220"
+		(property "Value" "150"
 			(at 180.34 43.434 0)
 			(show_name no)
